Commit message: fixing position of base link

File: install/projekt/share/projekt/urdf/scara.urdf (robot description, URDF)
Before this commit: robot scara_robot, 8 links, 7 joints
Links:
- added link world
Joints:
- added joint world_to_base_footprint: type fixed, parent world, child base_footprint, origin xyz=$(arg base_x) $(arg base_y) $(arg base_z) rpy=0 0 $(arg base_yaw)
- joint table_camera_joint: parent base_link -> base_footprint

Commit message: image processing basics

File: install/projekt/share/projekt/urdf/scara.urdf (robot description, URDF)
Before this commit: robot scara_robot, 9 links, 8 joints
Joints:
- joint table_camera_joint: origin xyz=0.25 0.0 1.5 rpy=0 1.5707 0 -> xyz=0.25 0.0 1.0 rpy=0 1.5707 0
