Commit message: end effector red cube
end effector részben működik

File: projekt/urdf/scara.urdf (robot description, URDF)
Before this commit: robot scara_robot, 5 links, 4 joints
Links:
- added link red_cube_link; visual box size=0.01 0.01 0.01
Joints:
- added joint joint4: type fixed, parent end_effector, child red_cube_link, origin xyz=0.0 0.0 -0.1 rpy=0 0 0

Commit message: attach-detach system
működik a kocka end_effektorhoz ragasztása

File: projekt/urdf/scara.urdf (robot description, URDF)
Before this commit: robot scara_robot, 6 links, 5 joints
Links:
- removed link red_cube_link
- added link red_cube; visual box size=0.01 0.01 0.01
Joints:
- joint joint4: child red_cube_link -> red_cube

Commit message: camera visual, image not working yet
már van egy asztal feletti kamera

File: projekt/urdf/scara.urdf (robot description, URDF)
Before this commit: robot scara_robot, 6 links, 5 joints
Links:
- added link table_camera_link, mass 1.0e-03; visual box size=.05 .05 .05
- added link table_camera_link_optical
Joints:
- added joint table_camera_joint: type fixed, parent base_link, child table_camera_link, origin xyz=0.25 0.0 1.5 rpy=0 0 0
- added joint table_camera_optical_joint: type fixed, parent table_camera_link, child table_camera_link_optical, origin xyz=0 0 0 rpy=-1.5707 0 -1.5707

Commit message: sorting node implementation

File: projekt/urdf/scara.urdf (robot description, URDF)
Before this commit: robot scara_robot, 9 links, 8 joints
Links:
- link end_effector: geometry collision cylinder length=0.02 radius=0.018; visual cylinder length=0.3 radius=0.02
